File: sun_sensor.kicad_sch (KiCad schematic)
At the start: 0 parts

Commit message: Add XYZ photodiodes to sun sensor. Fix hierarchical labels on MCU.
Parts:
- added C27, C28, C29, C30, C31, C32: 10nF, Capacitor_SMD:C_0603_1608Metric, symbol Device:C
- added R15, R16, R17, R18, R19, R20: 1k, Resistor_SMD:R_0603_1608Metric, symbol Device:R
- added RXN_LOAD, RXP_LOAD, RYN_LOAD, RYP_LOAD, RZN_LOAD, RZP_LOAD: 10k, Resistor_SMD:R_0603_1608Metric, symbol Device:R
- added SUN_XN, SUN_XP, SUN_YN, SUN_YP, SUN_ZN, SUN_ZP: TEMD7000X01, TEMD7000X01:XDCR_TEMD7000X01, symbol TEMD7000X01:TEMD7000X01
Connections:
- new net GND: C27.1, C28.1, C29.1, C30.1, C31.1, C32.1, RXN_LOAD.2, RXP_LOAD.2, RYN_LOAD.2, RYP_LOAD.2, RZN_LOAD.2, RZP_LOAD.2, SUN_XN.A, SUN_XP.A, SUN_YN.A, SUN_YP.A, SUN_ZN.A, SUN_ZP.A
- new net SUN_XN_ADC: C28.2, R16.2
- new net SUN_XN_RAW: R16.1, RXN_LOAD.1, SUN_XN.C
- new net SUN_XP_ADC: C27.2, R15.2
- new net SUN_XP_RAW: R15.1, RXP_LOAD.1, SUN_XP.C
- new net SUN_YN_ADC: C30.2, R18.2
- new net SUN_YN_RAW: R18.1, RYN_LOAD.1, SUN_YN.C
- new net SUN_YP_ADC: C29.2, R17.2
- new net SUN_YP_RAW: R17.1, RYP_LOAD.1, SUN_YP.C
- new net SUN_ZN_ADC: C32.2, R20.2
- new net SUN_ZN_RAW: R20.1, RZN_LOAD.1, SUN_ZN.C
- new net SUN_ZP_ADC: C31.2, R19.2
- new net SUN_ZP_RAW: R19.1, RZP_LOAD.1, SUN_ZP.C
